File: InGaAs_General_PD_v0.1/InGaAs_General_PD_v0.1.kicad_sch (KiCad schematic)
At the start: 48 parts, among them J1 C914558-SMA-KE-P903, J2 C914558-SMA-KE-P903, J3 2542-WR-3, U1 C1870618-OPA818IDRGR, U2 C2060224-OPA211AIDRGR, U3 C527498-OPA657U_2K5, U4 C42738-L78L05ABUTR, U5 C915681-L78L12ABUTR, U6 C157452-L79L05ABUTR, U7 C157399-L79L12ACUTR

Commit message: Commit Fixes
Parts:
- removed G1: IAMSnanofiber, IAMS:IAMSnanofiber, symbol IAMS:IAMSnanofiber
- removed G2: IAMS, IAMS:IAMS, symbol IAMS:IAMS
- removed G3: IAMSYb, IAMS:IAMSYb, symbol IAMS:IAMSYb
